File: ym2413-stereo-isa.kicad_pcb (KiCad board)
At the start: 2 copper layers, 119.4 x 98.7 mm, 78 parts, among them IC1 TEA2025B, IC10 LM7809_TO220, IC2 YM2413, IC3 YM2413, IC4 TL072, IC5 74LS245, IC6 74LS138, IC7 74LS32, IC8 74LS04, IC9 74LS74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

Commit message: Relocate volume pot and output jack; update gerbers; add CAD models
Parts:
- moved J2 21.5 mm to (190.8, 94.5)
- moved C43 7.37 mm to (190.2, 74.2)
- moved C18 7.10 mm to (176.0, 75.8), turned to -90 degrees
- moved C17 6.50 mm to (145.0, 77.3), turned to -90 degrees
- moved R15 5.08 mm to (176.1, 57.7), turned to -90 degrees
- moved C39 4.88 mm to (179.1, 104.2), turned to -90 degrees
- moved RV1 3.96 mm to (188.4, 57.1), turned to 90 degrees
- moved C36 0.13 mm to (179.1, 101.5)
Routing:
- net Net-(J2-Pad2): track 7.28 -> 28.2 mm
- net Net-(J2-Pad3): track 5.56 -> 24.0 mm
- net GNDA: track 97.6 -> 84.4 mm
- net Net-(C18-Pad1): track 49.9 -> 36.9 mm
- net Net-(C17-Pad1): track 61.8 -> 53.9 mm
- net Net-(C11-Pad2): track 17.3 -> 22.4 mm
- net Net-(IC1-Pad10): track 12.3 -> 16.7 mm
- net Net-(IC1-Pad7): track 11.5 -> 15.1 mm
- net Net-(C10-Pad2): track 21.6 -> 19.7 mm
- net Net-(IC1-Pad3): track 28.4 -> 26.8 mm
