File: ym2413-stereo-isa.kicad_pcb (KiCad board)
At the start: 2 copper layers, 119.4 x 98.7 mm, 78 parts, among them IC1 TEA2025B, IC10 LM7809_TO220, IC2 YM2413, IC3 YM2413, IC4 TL072, IC5 74LS245, IC6 74LS138, IC7 74LS32, IC8 74LS04, IC9 74LS74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

Commit message: correct capacitor footprint; move voltage divider; flip coupling caps
Parts:
- C1, C6: value 100uF 16V -> 10uF 16V
- R1, R10, R11, R12, R13, R14, R15, R16, R17, R18, R2, R3, R4, R5, R6, R7, R8, R9: footprint Resistor_THT:R_Axial_DIN0204_L3.6mm_D1.6mm_P5.08mm_Horizontal -> Resistor_THT:R_Axial_DIN0207_L6.3mm_D2.5mm_P7.62mm_Horizontal
- moved R13 3.18 mm to (158.5, 65.2)
- moved R5 3.05 mm to (135.3, 40.5)
- moved R1 2.94 mm to (116.6, 55.2)
- moved C18 2.48 mm to (176.0, 78.2), turned to 90 degrees
- moved C17 2.40 mm to (145.0, 79.7), turned to 90 degrees
- moved R3 2.18 mm to (134.4, 55.2)
- moved R2 1.78 mm to (117.7, 40.5)
- moved R17 1.78 mm to (149.4, 88.0)
- moved R18 1.65 mm to (169.7, 87.9)
- moved R14 1.38 mm to (158.6, 47.8)
- moved R16 1.29 mm to (176.8, 47.8)
- moved C28 1.14 mm to (149.3, 68.3)
- moved C29 1.14 mm to (156.6, 68.3)
- moved R7 0.89 mm to (144.0, 60.4)
- moved R8 0.89 mm to (143.9, 44.7)
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Connections:
- C17 pad 2: Net-(IC1-Pad10) -> Net-(C17-Pad2)
- C18 pad 2: Net-(IC1-Pad7) -> Net-(C18-Pad2)
- IC1 pad 10: Net-(IC1-Pad10) -> Net-(C17-Pad1)
- IC1 pad 7: Net-(IC1-Pad7) -> Net-(C18-Pad1)
- R15 pad 1: Net-(C17-Pad1) -> Net-(C17-Pad2)
- R16 pad 1: Net-(C18-Pad1) -> Net-(C18-Pad2)
- R4 pad 1: Net-(R1-Pad1) -> /RO_L
- R6 pad 1: Net-(R10-Pad2) -> /RO_R
- R7 pad 1: Net-(R1-Pad1) -> /MO_L
- R8 pad 1: Net-(R10-Pad2) -> /MO_R
- RV1 pad 3A: Net-(C17-Pad1) -> Net-(C17-Pad2)
- RV1 pad 3B: Net-(C18-Pad1) -> Net-(C18-Pad2)
Routing:
- net Net-(C17-Pad2): track 0.00 -> 50.3 mm
- net Net-(C17-Pad1): track 53.9 -> 13.2 mm
- net Net-(C18-Pad2): track 0.00 -> 36.3 mm
- net /RO_L: track 3.93 -> 30.9 mm, vias 0 -> 1
- net /MO_L: track 3.93 -> 26.3 mm, vias 0 -> 1
- net Net-(C18-Pad1): track 36.9 -> 15.1 mm
- net /MO_R: track 3.30 -> 21.4 mm
- net /RO_R: track 3.30 -> 21.1 mm
- net Net-(IC1-Pad10): track 16.7 -> 0.00 mm
- net Net-(IC1-Pad7): track 15.1 -> 0.00 mm
- net GNDA: track 84.4 -> 76.6 mm
- net Net-(R10-Pad2): track 28.8 -> 21.2 mm
- net Net-(R1-Pad1): track 29.3 -> 21.9 mm
- net Net-(C23-Pad1): track 6.48 -> 0.00 mm
- net Net-(C10-Pad1): track 21.1 -> 25.0 mm
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