File: ym2413-stereo-isa.kicad_sch (KiCad schematic)
At the start: 78 parts, among them IC1 TEA2025B, IC10 LM7809_TO220, IC2 YM2413, IC3 YM2413, IC4 TL072, IC5 74LS245, IC6 74LS138, IC7 74LS32, IC8 74LS04, IC9 74LS74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

Commit message: correct capacitor footprint; move voltage divider; flip coupling caps
Parts:
- C1, C6: value 100uF 16V -> 10uF 16V
Connections:
- net MO_L: now also R7.1
- net MO_R: now also R8.1
- net RO_L: now also R4.1
- net RO_R: now also R6.1
- net at R16.1, RV1.3B: now also C18.2; no longer C18.1
- net at R10.2, R2.1, R5.1: no longer R6.1, R8.1
- net at R1.1, R3.1, R9.2: no longer R4.1, R7.1
- net at R15.1, RV1.3A: now also C17.2; no longer C17.1
- net at IC1.7 (IN.2(+)): now also C18.1; no longer C18.2
- net at IC1.10 (IN.1(+)): now also C17.1; no longer C17.2
Other:
- moved on the sheet: C17, C18, R3, R4, R5, R6, R7, R8
